File: powerOutput.kicad_sch (KiCad schematic)
At the start: 12 parts, among them J1 Screw_Terminal_01x08, J9 Screw_Terminal_01x08, K1 SANYOU_SRD-S-124D, K2 SANYOU_SRD-S-124D, K3 SANYOU_SRD-S-124D, K4 SANYOU_SRD-S-124D, U4 ULN2803CDW, U7 ULN2803CDW

Commit message: almost done
Connections:
- net 230V: now reaches J1.2 (Pin_2), K1.3
- net 230V: now also J1.3 (Pin_3), J1.4 (Pin_4), J1.5 (Pin_5), K2.3, K3.3, K4.3
Other:
- moved on the sheet: J1, K1, K2, K3, K4, TP1, TP2, TP3, TP4
