File: controesp.kicad_pcb (KiCad board)
At the start: 2 copper layers, 216.9 x 86.5 mm, 75 parts, among them J1 Screw_Terminal_01x08, J13 Conn_01x19_Socket, J14 Conn_01x16_Socket, J15 Screw_Terminal_01x02, J16 Conn_01x19_Socket, J17 Conn_01x19_Socket, J2 Screw_Terminal_01x04, J3 Conn_01x14_Socket, J4 Conn_01x14_Pin, J5 Conn_01x16_Pin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

Commit message: splitted hat pcb into seperate proj
Parts:
- removed C1, C2, C4: 100nF, Capacitor_SMD:C_0805_2012Metric_Pad1.18x1.45mm_HandSolder
- removed C5: SMD TAN.10/35, Capacitor_SMD:C_0805_2012Metric_Pad1.18x1.45mm_HandSolder
- removed the G*** at (237.7, 109.2)
- removed J13, J16, J17: Conn_01x19_Socket, Connector_PinSocket_2.54mm:PinSocket_1x19_P2.54mm_Vertical
- removed J4: Conn_01x14_Pin, Connector_PinHeader_2.54mm:PinHeader_1x14_P2.54mm_Vertical
- removed J5: Conn_01x16_Pin, Connector_PinHeader_2.54mm:PinHeader_1x16_P2.54mm_Vertical
- removed R11, R12, R13: 0, Resistor_SMD:R_0805_2012Metric_Pad1.20x1.40mm_HandSolder
- removed R14, R15, R16, R17: 10k, Resistor_SMD:R_0805_2012Metric_Pad1.20x1.40mm_HandSolder
- removed U3: TCA9517ADGK, Package_SO:VSSOP-8_3x3mm_P0.65mm
- removed U9: PCF8575DBR, Package_SO:SSOP-24_5.3x8.2mm_P0.65mm
Routing:
- net /controesp_hat/GND: track 266.4 -> 0.00 mm, vias 5 -> 0
- net /controesp_hat/VCC: track 115.5 -> 0.00 mm, vias 2 -> 0
- net /controesp_hat/3V3: track 102.6 -> 0.00 mm, vias 2 -> 0
- net /controesp_hat/SCL_5V: track 84.2 -> 0.00 mm, vias 4 -> 0
- net /controesp_hat/SDA_5V: track 80.4 -> 0.00 mm, vias 2 -> 0
- net /controesp_hat/RX2: track 70.4 -> 0.00 mm, vias 2 -> 0
- net /controesp_hat/TX2: track 67.5 -> 0.00 mm, vias 2 -> 0
- net /controesp_hat/13: track 58.3 -> 0.00 mm
- net /controesp_hat/32: track 49.7 -> 0.00 mm, vias 3 -> 0
- net /controesp_hat/33: track 48.5 -> 0.00 mm, vias 3 -> 0
- net /controesp_hat/14: track 47.6 -> 0.00 mm
- net /controesp_hat/26: track 47.0 -> 0.00 mm, vias 1 -> 0
- net /controesp_hat/P15: track 46.9 -> 0.00 mm
- net /controesp_hat/25: track 45.9 -> 0.00 mm, vias 1 -> 0
- net /controesp_hat/27: track 43.7 -> 0.00 mm
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- removed copper zone on B.Cu, net /controesp_hat/GND
- removed copper zone on F.Cu, net /controesp_hat/GND
Other:
- board size 216.9 x 86.5 mm -> 103 x 86.5 mm
- board text removed: "controesp.hat - rev 1"
